File: split_65/split_65.sch (KiCad schematic (older format))
At the start: 156 parts, among them SW1 SW_Push, SW10 SW_Push, SW11 SW_Push, SW12 SW_Push, SW13 SW_Push, SW14 SW_Push, SW15 SW_Push, SW16 SW_Push, SW17 SW_Push, SW18 SW_Push, SW19 SW_Push, SW2 SW_Push, SW20 SW_Push, SW21 SW_Push, SW22 SW_Push, SW23 SW_Push, SW24 SW_Push, SW25 SW_Push, SW26 SW_Push, SW27 SW_Push, SW28 SW_Push, SW29 SW_Push, SW3 SW_Push, SW30 SW_Push, SW31 SW_Push, SW32 SW_Push, SW33 SW_Push, SW34 SW_Push, SW35 SW_Push, SW36 SW_Push, SW37 SW_Push, SW38 SW_Push, SW39 SW_Push, SW4 SW_Push, SW40 SW_Push, SW41 SW_Push, SW42 SW_Push, SW43 SW_Push, SW44 SW_Push, SW45 SW_Push, SW46 SW_Push, SW47 SW_Push, SW48 SW_Push, SW49 SW_Push, SW5 SW_Push, SW50 SW_Push, SW51 SW_Push, SW52 SW_Push, SW53 SW_Push, SW54 SW_Push, SW55 SW_Push, SW56 SW_Push, SW57 SW_Push, SW58 SW_Push, SW59 SW_Push, SW6 SW_Push, SW60 SW_Push, SW61 SW_Push, SW62 SW_Push, SW63 SW_Push, SW64 SW_Push, SW65 SW_Push, SW66 SW_Push, SW67 SW_Push, SW68 SW_Push, SW69 SW_Push, SW7 SW_Push, SW70 SW_Push, SW71 SW_Push, SW72 SW_Push, SW73 SW_Push, SW74 SW_Push, SW75 SW_Push, SW76 SW_Push, SW77 SW_Push, SW78 SW_Push, SW79 SW_Push, SW8 SW_Push, SW80 SW_Push, SW81 SW_Push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

Commit message: setup schematic hierarchies, update images
Parts:
- removed D1, D10, D11, D12, D13, D14, D15, D16, D17, D18, D19, D2, D20, D21, D22, D23, D24, D25, D26, D27, D28, D29, D3, D30, D31, D32, D33, D34, D35, D36, D37, D38, D39, D4, D40, D41, D42, D43, D44, D45, D46, D47, D48, D49, D5, D50, D51, D52, D53, D54, D55, D56, D57, D58, D59, D6, D60, D61, D62, D63, D64, D65, D66, D67, D68, D69, D7, D70, D71, D72, D73, D74, D8, D9: D_Small, Diode_SMD:D_0603_1608Metric_Pad1.05x0.95mm_HandSolder, symbol Device:D_Small
- removed SW1, SW12, SW13, SW14, SW15, SW18, SW19, SW2, SW20, SW21, SW23, SW24, SW25, SW26, SW29, SW3, SW30, SW31, SW32, SW33, SW34, SW35, SW36, SW37, SW38, SW39, SW4, SW40, SW41, SW44, SW45, SW46, SW47, SW48, SW49, SW5, SW50, SW51, SW53, SW54, SW55, SW56, SW59, SW60, SW61, SW62, SW65, SW66, SW67, SW69, SW70, SW71, SW72, SW76, SW77, SW78, SW79, SW80, SW81, SW82: SW_Push, MX_Alps_Hybrid:MXOnly-1U-NoLED, symbol Switch:SW_Push
- removed SW10, SW16, SW22, SW52, SW57, SW63: SW_Push, MX_Alps_Hybrid:MXOnly-1.25U-NoLED, symbol Switch:SW_Push
- removed SW11, SW17, SW58, SW6, SW64, SW74: SW_Push, MX_Alps_Hybrid:MXOnly-1.5U-NoLED, symbol Switch:SW_Push
- removed SW27: SW_Push, MX_Alps_Hybrid:MXOnly-2.75U-NoLED, symbol Switch:SW_Push
- removed SW28, SW43: SW_Push, MX_Alps_Hybrid:MXOnly-3U-NoLED, symbol Switch:SW_Push
- removed SW42, SW75, SW9: SW_Push, MX_Alps_Hybrid:MXOnly-2.25U-NoLED, symbol Switch:SW_Push
- removed SW68: SW_Push, MX_Alps_Hybrid:MXOnly-1.75U-NoLED, symbol Switch:SW_Push
- removed SW7: SW_Push, MX_Alps_Hybrid:MXOnly-1.75U, symbol Switch:SW_Push
- removed SW73: SW_Push, MX_Alps_Hybrid:MXOnly-2U-NoLED, symbol Switch:SW_Push
- removed SW8: SW_Push, MX_Alps_Hybrid:MXOnly-1.25U, symbol Switch:SW_Push
Connections:
- wire segments 157 -> 0
