File: pcb/split_65.kicad_pcb (KiCad board)
At the start: 2 copper layers, 375 x 105.4 mm, 335 parts, among them J1 PJ-3200B-4A, J10 AVR-ISP-6, J11 Breakaway_Tabs, J12 Breakaway_Tabs, J13 Breakaway_Tabs, J14 Breakaway_Tabs, J15 Breakaway_Tabs, J16 Breakaway_Tabs, J2 AVR-ISP-6, J3 Breakaway_Tabs, J4 Breakaway_Tabs, J5 Breakaway_Tabs, J6 Breakaway_Tabs, J7 Breakaway_Tabs, J8 Breakaway_Tabs, J9 PJ-3200B-4A, Q1 2N7002, Q2 2N7002, SW1 SW_Push, SW2 SW_Push, U1 ATmega32U4-AU, U2 PRTR5V0U2X, U3 ATmega32U4-AU, U4 PRTR5V0U2X, Y1 16MHz, Y2 16MHz

Commit message: added rgb underglow and step files
Parts:
- removed R91, R92: 10k, Resistor_SMD:R_0805_2012Metric
- LED1, LED10, LED11, LED12, LED13, LED14, LED15, LED16, LED2, LED3, LED4, LED5, LED6, LED7, LED8, LED9: value WS2812B -> VAL**
- MX0, MX1, MX10, MX11, MX12, MX13, MX14, MX15, MX18, MX19, MX2, MX20, MX21, MX22, MX23, MX25, MX26, MX27, MX28, MX29, MX3, MX30, MX38, MX39, MX4, MX40, MX41, MX42, MX43, MX44, MX46, MX47, MX48, MX49, MX5, MX50, MX51, MX52, MX53, MX54, MX56, MX57, MX58, MX59, MX6, MX60, MX61, MX62, MX64, MX65, MX66, MX67, MX68, MX69, MX7, MX71, MX72, MX8, MX80, MX81, MX82: value MXOnly-1U -> 1U
- moved SW1 267.7 mm to (72.6, 100.0), turned to 0 degrees
- moved LED7 218.4 mm to (38.1, 71.4), turned to 90 degrees
- moved C28 212.1 mm to (378.6, 75.6)
- moved LED14 210.2 mm to (378.6, 71.4), turned to 270 degrees
- moved C1 200.3 mm to (57.6, 121.5), turned to 45 degrees
- moved C29 198.6 mm to (378.6, 104.8)
- moved LED15 198.1 mm to (378.6, 100.0), turned to 270 degrees
- moved LED1 195.3 mm to (38.1, 128.6), turned to 270 degrees
- moved C3 193.6 mm to (45.7, 109.8)
- moved C30 192.4 mm to (378.6, 133.4)
- moved C2 190.5 mm to (57.5, 116.7), turned to 315 degrees
- moved C21 189.3 mm to (38.1, 75.3)
- moved LED8 188.7 mm to (38.1, 100.0), turned to 270 degrees
- moved C22 175.5 mm to (38.1, 103.9)
- moved C15 173.2 mm to (37.2, 132.5)
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Connections:
- LED11 pad 4: Net-(LED11-Pad4) -> Net-(LED10-Pad2)
- LED12 pad 4: Net-(LED10-Pad2) -> Net-(LED11-Pad2)
- LED13 pad 4: Net-(LED11-Pad2) -> Net-(LED12-Pad2)
- LED14 pad 4: Net-(LED12-Pad2) -> Net-(LED13-Pad2)
- LED15 pad 2: Net-(LED10-Pad4) -> Net-(LED15-Pad2)
- LED15 pad 4: Net-(LED13-Pad2) -> Net-(LED14-Pad2)
- LED16 pad 4: Net-(LED14-Pad2) -> Net-(LED15-Pad2)
- LED2 pad 4: Net-(LED2-Pad4) -> Net-(LED1-Pad2)
- LED3 pad 4: Net-(LED1-Pad2) -> Net-(LED2-Pad2)
- LED4 pad 4: Net-(LED2-Pad2) -> Net-(LED3-Pad2)
- LED5 pad 4: Net-(LED3-Pad2) -> Net-(LED4-Pad2)
- LED6 pad 4: Net-(LED4-Pad2) -> Net-(LED5-Pad2)
- LED7 pad 2: Net-(LED2-Pad4) -> Net-(LED7-Pad2)
- LED7 pad 4: Net-(LED5-Pad2) -> Net-(LED6-Pad2)
- LED8 pad 4: Net-(LED6-Pad2) -> Net-(LED7-Pad2)
- LED9 pad 2: Net-(LED11-Pad4) -> Net-(LED10-Pad4)
- SW1 pad 2: Net-(R91-Pad1) -> RESET
- SW2 pad 2: Net-(R92-Pad1) -> RESET-R
- U1 pad 13: Net-(R91-Pad1) -> RESET
- U3 pad 13: Net-(R92-Pad1) -> RESET-R
Routing:
- net LEDGND: track 504.6 -> 0.00 mm, vias 6 -> 0
- net +5V: track 332.0 -> 6.23 mm
- net ROW2: track 125.1 -> 0.00 mm, vias 2 -> 0
- net ROW1: track 120.3 -> 0.00 mm, vias 2 -> 0
- net ROW4: track 115.5 -> 5.36 mm
- net COL5: track 93.0 -> 0.00 mm
- net ROW0: track 90.7 -> 0.00 mm, vias 2 -> 0
- net GND: track 149.2 -> 71.9 mm
- net COL4: track 69.7 -> 0.00 mm
- net COL6: track 69.7 -> 0.00 mm
- net COL7: track 69.6 -> 0.00 mm
- net ROW3: track 65.6 -> 0.00 mm
- net D+: track 70.2 -> 4.97 mm
- net D-: track 70.2 -> 5.15 mm
- net COL0: track 59.5 -> 0.00 mm
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Other:
- outline, holes or cut-outs redrawn

Commit message: more traces
Changed lines of the file:
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@@
   )
   (setup
-    (last_trace_width 0.55)
+    (last_trace_width 0.254)
     (user_trace_width 0.254)
     (user_trace_width 0.381)
@@
     (fp_line (start -0.8 0.4) (end 0.8 0.4) (layer B.Fab) (width 0.1))
     (fp_line (start -0.8 -0.4) (end -0.8 0.4) (layer B.Fab) (width 0.1))
-    (pad 2 smd roundrect (at 0.7875 0 45) (size 0.875 0.95) (layers B.Cu B.Paste B.Mask) (roundrect_rratio 0.25)
+    (pad 2 smd roundrect (at 0.787501 0 45) (size 0.875 0.95) (layers B.Cu B.Paste B.Mask) (roundrect_rratio 0.25)
       (net 1 GND))
-    (pad 1 smd roundrect (at -0.7875 0 45) (size 0.875 0.95) (layers B.Cu B.Paste B.Mask) (roundrect_rratio 0.25)
+    (pad 1 smd roundrect (at -0.787501 0 45) (size 0.875 0.95) (layers B.Cu B.Paste B.Mask) (roundrect_rratio 0.25)
       (net 2 "Net-(C1-Pad1)"))
     (model ${KISYS3DMOD}/Capacitor_SMD.3dshapes/C_0603_1608Metric.wrl
@@
     (polygon
       (pts
-        (xy 63.10339 123.82552) (xy 63.10339 114.30048) (xy 52.38772 114.30048) (xy 52.38772 123.82552)
+        (xy 63.10339 123.82552) (xy 63.10339 114.30048) (xy 53.57835 114.30048) (xy 53.57835 123.82552)
       )
     )

Commit message: generated step files
Parts:
- moved R24 22.7 mm to (44.1, 128.6), turned to 90 degrees
Routing:
- net Net-(U1-Pad1): track 0.00 -> 6.85 mm
