File: pcb/split_65.sch (KiCad schematic (older format))
At the start: 312 parts, among them J1 PJ-3200B-4A, J10 AVR-ISP-6, J11 Breakaway_Tabs, J12 Breakaway_Tabs, J13 Breakaway_Tabs, J14 Breakaway_Tabs, J15 Breakaway_Tabs, J16 Breakaway_Tabs, J2 AVR-ISP-6, J3 Breakaway_Tabs, J4 Breakaway_Tabs, J5 Breakaway_Tabs, J6 Breakaway_Tabs, J7 Breakaway_Tabs, J8 Breakaway_Tabs, J9 PJ-3200B-4A, Q1 2N7002, Q2 2N7002, SW1 SW_Push, SW2 SW_Push, U1 ATmega32U4-AU, U2 PRTR5V0U2X, U3 ATmega32U4-AU, U4 PRTR5V0U2X, Y1 16MHz, Y2 16MHz

Commit message: laid out diodes and resistors
Parts:
- removed MH1, MH2: HOLE, MountingHole:MountingHole_5mm, symbol Connector_Generic:Conn_01x01
Connections:
- no-connect marks 20 -> 18
Other:
- note removed: "Passthrough Holes"
- note removed: "Passthrough Holes\n"
Changed lines of the file:
@@
 EESchema Schematic File Version 4
+LIBS:split_65-cache
 EELAYER 26 0
 EELAYER END
@@
 	5650 6400 9175 6400
 Wire Notes Line
-	9175 12825 9175 15275
-Wire Notes Line
 	5650 13975 9175 13975
-Text Notes 7775 12925 0    50   ~ 0
-Passthrough Holes\n
-Text Notes 7775 5350 0    50   ~ 0
-Passthrough Holes
-$Comp
-L Connector_Generic:Conn_01x01 MH1
-U 1 1 5C5F2D6B
-P 8150 5600
-F 0 "MH1" H 8229 5642 50  0000 L CNN
-F 1 "HOLE" H 8229 5551 50  0000 L CNN
-F 2 "MountingHole:MountingHole_5mm" H 8150 5600 50  0001 C CNN
-F 3 "~" H 8150 5600 50  0001 C CNN
-	1    8150 5600
-	1    0    0    -1
-$EndComp
-NoConn ~ 7950 5600
-$Comp
-L Connector_Generic:Conn_01x01 MH2
-U 1 1 5C7F1ECF
-P 8175 13150
-F 0 "MH2" H 8254 13192 50  0000 L CNN
-F 1 "HOLE" H 8254 13101 50  0000 L CNN
-F 2 "MountingHole:MountingHole_5mm" H 8175 13150 50  0001 C CNN
-F 3 "~" H 8175 13150 50  0001 C CNN
-	1    8175 13150
-	1    0    0    -1
-$EndComp
-NoConn ~ 7975 13150
 Text Notes 7775 6500 0    50   ~ 0
 Half Detection
@@
 Connection ~ 9550 4225
 Wire Wire Line
-	10125 4025 10425 4025
-Wire Wire Line
 	9775 4075 9775 4925
-Connection ~ 10425 4025
-Wire Wire Line
-	10075 4075 10375 4075
-Wire Wire Line
-	9975 4175 10275 4175
-Connection ~ 10275 4175
-Wire Wire Line
-	9925 4225 10150 4225
-Connection ~ 10150 4225
 Wire Wire Line
 	9375 4175 9675 4175
@@
 L MX_Alps_Hybrids:MX-1U MX33
 U 1 1 5CCB75DC
-P 9950 4050
-F 0 "MX33" H 10036 4267 60  0000 C CNN
-F 1 "MXOnly-1U" H 10036 4193 20  0000 C CNN
-F 2 "MX_Alps_Hybrid:MXOnly-1.5U" H 9925 4025 60  0001 C CNN
-F 3 "" H 9925 4025 60  0001 C CNN
-	1    9950 4050
+P 10550 4050
+F 0 "MX33" H 10636 4267 60  0000 C CNN
+F 1 "MXOnly-1U" H 10636 4193 20  0000 C CNN
+F 2 "MX_Alps_Hybrid:MXOnly-1.5U" H 10525 4025 60  0001 C CNN
+F 3 "" H 10525 4025 60  0001 C CNN
+	1    10550 4050
 	1    0    0    -1
 $EndComp
@@
 	3400 12225 3500 12225
 Connection ~ 3400 12225
+Wire Notes Line
+	9175 12825 9175 15275
+Wire Wire Line
+	10725 4025 11025 4025
+Connection ~ 11025 4025
+Wire Wire Line
+	10675 4075 10975 4075
+Wire Wire Line
+	10575 4175 10875 4175
+Connection ~ 10875 4175
+Wire Wire Line
+	10525 4225 10750 4225
+Connection ~ 10750 4225
 $EndSCHEMATC

Commit message: add switch, edit models
Parts:
- removed D34, D35, D36, D79, D80, D81: LED_3mm, locallib:LED_D3.0mm, symbol Device:LED_Small
- removed R38, R39, R40, R89, R90, R91: 1k, Resistor_SMD:R_0805_2012Metric, symbol Device:R_Small
- added D0: SOD-123, Diode_SMD:D_SOD-123, symbol Device:D_Small
- added MX0: MXOnly-1U, MX_Alps_Hybrid:MXOnly-1U, symbol MX_Alps_Hybrids:MX-1U
- added R0: 470, Resistor_SMD:R_0805_2012Metric, symbol Device:R_Small
- renumbered D37 to D34, D38 to D35, D39 to D36, D40 to D37, D41 to D38, D42 to D39, D43 to D40, D44 to D41, D45 to D42, D46 to D43, D47 to D44, D48 to D45, D49 to D46, D50 to D47, D51 to D48, D52 to D49, D53 to D50, D54 to D51, D55 to D52, D56 to D53, D57 to D54, D58 to D55, D59 to D56, D60 to D57, D61 to D58, D62 to D59, D63 to D60, D64 to D61, D65 to D62, D66 to D63, D67 to D64, D68 to D65, D69 to D66, D70 to D67, D71 to D68, D72 to D69, D73 to D70, D74 to D71, D75 to D72, D76 to D73, D77 to D74, D78 to D75, D82 to D76, MX34 to MX33, MX33 to MX34, R41 to R38, R42 to R39, R43 to R40, R44 to R41, R45 to R42, R46 to R43, R47 to R44, R48 to R45, R49 to R46, R50 to R47, R51 to R48, R52 to R49, R53 to R50, R54 to R51, R55 to R52, R56 to R53, R57 to R54, R58 to R55, R59 to R56, R60 to R57, R61 to R58, R62 to R59, R63 to R60, R64 to R61, R65 to R62, R66 to R63, R67 to R64, R68 to R65, R69 to R66, R70 to R67, R71 to R68, R72 to R69, R73 to R70, R74 to R71, R75 to R72, R76 to R73, R77 to R74, R78 to R75, R79 to R76, R80 to R77, R81 to R78, R82 to R79, R83 to R80, R84 to R81, R85 to R82, R86 to R83, R87 to R84, R88 to R85, R92 to R86, R93 to R87, R94 to R88, R95 to R89, R96 to R90
Connections:
- net labels added: COL7
- net labels removed: LEDIND-1, LEDIND-1-R, LEDIND-2, LEDIND-2-R, LEDIND-3, LEDIND-3-R
- wire segments 687 -> 670
Other:
- note removed: "Indicator LEDs\n"

Commit message: add resistor to rst, rgb underglow
Parts:
- added C15, C16, C17, C18, C19, C20, C21, C22, C23, C24, C25, C26, C27, C28, C29, C30: 0.1uF, Capacitor_SMD:C_0603_1608Metric, symbol Device:C_Small
- added LED1, LED10, LED11, LED12, LED13, LED14, LED15, LED16, LED2, LED3, LED4, LED5, LED6, LED7, LED8, LED9: WS2812B, WS2812B:WS2812B, symbol ws2812b:WS2812B
- added R? (x2): 10k, Resistor_SMD:R_0805_2012Metric, symbol Device:R_Small
Connections:
- net labels added: RGBLED, RGBLED-R
- wire segments 670 -> 809
- no-connect marks 18 -> 20

Commit message: added rgb underglow and step files
Parts:
- removed R? (x2): 10k, Resistor_SMD:R_0805_2012Metric, symbol Device:R_Small
- added R91, R92: 470, Resistor_SMD:R_0805_2012Metric, symbol Device:R_Small
- renumbered LED11 to LED10, LED13 to LED11, LED15 to LED12, LED10 to LED13, LED12 to LED14, LED14 to LED15, LED3 to LED2, LED5 to LED3, LED7 to LED4, LED2 to LED5, LED4 to LED6, LED6 to LED7
Connections:
- wire segments 809 -> 811
Changed lines of the file:
@@
 	1    0    0    -1
 $EndComp
-Wire Wire Line
-	2325 8925 2625 8925
 $Comp
 L Device:D_Schottky_Small D34
@@
 	2900 13950 3000 13950
 $Comp
-L ws2812b:WS2812B LED3
+L ws2812b:WS2812B LED2
 U 1 1 5CD644FA
 P 15700 2475
-F 0 "LED3" H 15700 2962 60  0000 C CNN
+F 0 "LED2" H 15700 2962 60  0000 C CNN
 F 1 "WS2812B" H 15700 2856 60  0000 C CNN
 F 2 "WS2812B:WS2812B" V 15650 2475 60  0001 C CNN
@@
 $EndComp
 $Comp
-L ws2812b:WS2812B LED5
+L ws2812b:WS2812B LED3
 U 1 1 5CDE9D22
 P 15700 3350
-F 0 "LED5" H 15700 3837 60  0000 C CNN
+F 0 "LED3" H 15700 3837 60  0000 C CNN
 F 1 "WS2812B" H 15700 3731 60  0000 C CNN
 F 2 "WS2812B:WS2812B" V 15650 3350 60  0001 C CNN
@@
 $EndComp
 $Comp
-L ws2812b:WS2812B LED7
+L ws2812b:WS2812B LED4
 U 1 1 5CDE9D29
 P 15700 4225
-F 0 "LED7" H 15700 4712 60  0000 C CNN
+F 0 "LED4" H 15700 4712 60  0000 C CNN
 F 1 "WS2812B" H 15700 4606 60  0000 C CNN
 F 2 "WS2812B:WS2812B" V 15650 4225 60  0001 C CNN
@@
 $EndComp
 $Comp
-L ws2812b:WS2812B LED2
+L ws2812b:WS2812B LED5
 U 1 1 5CEF2414
 P 17425 1600
-F 0 "LED2" H 17425 2087 60  0000 C CNN
+F 0 "LED5" H 17425 2087 60  0000 C CNN
 F 1 "WS2812B" H 17425 1981 60  0000 C CNN
 F 2 "WS2812B:WS2812B" V 17375 1600 60  0001 C CNN
@@
 $EndComp
 $Comp
-L ws2812b:WS2812B LED4
+L ws2812b:WS2812B LED6
 U 1 1 5CEF241B
 P 17425 2475
-F 0 "LED4" H 17425 2962 60  0000 C CNN
+F 0 "LED6" H 17425 2962 60  0000 C CNN
 F 1 "WS2812B" H 17425 2856 60  0000 C CNN
 F 2 "WS2812B:WS2812B" V 17375 2475 60  0001 C CNN
@@
 $EndComp
 $Comp
-L ws2812b:WS2812B LED6
+L ws2812b:WS2812B LED7
 U 1 1 5CEF2422
 P 17425 3350
-F 0 "LED6" H 17425 3837 60  0000 C CNN
+F 0 "LED7" H 17425 3837 60  0000 C CNN
 F 1 "WS2812B" H 17425 3731 60  0000 C CNN
 F 2 "WS2812B:WS2812B" V 17375 3350 60  0001 C CNN
@@
 Text GLabel 4175 1950 2    50   Input ~ 0
 RGBLED
-Text GLabel 16200 1400 2    50   Input ~ 0
+Text GLabel 16200 1200 2    50   Input ~ 0
 RGBLED
 Wire Wire Line
@@
 $EndComp
 $Comp
-L ws2812b:WS2812B LED11
+L ws2812b:WS2812B LED10
 U 1 1 5E78DF6D
 P 16450 10250
-F 0 "LED11" H 16450 10737 60  0000 C CNN
+F 0 "LED10" H 16450 10737 60  0000 C CNN
 F 1 "WS2812B" H 16450 10631 60  0000 C CNN
 F 2 "WS2812B:WS2812B" V 16400 10250 60  0001 C CNN
@@
 $EndComp
 $Comp
-L ws2812b:WS2812B LED13
+L ws2812b:WS2812B LED11
 U 1 1 5E78DF74
 P 16450 11125
-F 0 "LED13" H 16450 11612 60  0000 C CNN
+F 0 "LED11" H 16450 11612 60  0000 C CNN
 F 1 "WS2812B" H 16450 11506 60  0000 C CNN
 F 2 "WS2812B:WS2812B" V 16400 11125 60  0001 C CNN
@@
 $EndComp
 $Comp
-L ws2812b:WS2812B LED15
+L ws2812b:WS2812B LED12
 U 1 1 5E78DF7B
 P 16450 12000
-F 0 "LED15" H 16450 12487 60  0000 C CNN
+F 0 "LED12" H 16450 12487 60  0000 C CNN
 F 1 "WS2812B" H 16450 12381 60  0000 C CNN
 F 2 "WS2812B:WS2812B" V 16400 12000 60  0001 C CNN
@@
 $EndComp
 $Comp
-L ws2812b:WS2812B LED10
+L ws2812b:WS2812B LED13
 U 1 1 5E78DF82
 P 18175 9375
-F 0 "LED10" H 18175 9862 60  0000 C CNN
+F 0 "LED13" H 18175 9862 60  0000 C CNN
 F 1 "WS2812B" H 18175 9756 60  0000 C CNN
 F 2 "WS2812B:WS2812B" V 18125 9375 60  0001 C CNN
@@
 $EndComp
 $Comp
-L ws2812b:WS2812B LED12
+L ws2812b:WS2812B LED14
 U 1 1 5E78DF89
 P 18175 10250
-F 0 "LED12" H 18175 10737 60  0000 C CNN
+F 0 "LED14" H 18175 10737 60  0000 C CNN
 F 1 "WS2812B" H 18175 10631 60  0000 C CNN
 F 2 "WS2812B:WS2812B" V 18125 10250 60  0001 C CNN
@@
 $EndComp
 $Comp
-L ws2812b:WS2812B LED14
+L ws2812b:WS2812B LED15
 U 1 1 5E78DF90
 P 18175 11125
-F 0 "LED14" H 18175 11612 60  0000 C CNN
+F 0 "LED15" H 18175 11612 60  0000 C CNN
 F 1 "WS2812B" H 18175 11506 60  0000 C CNN
 F 2 "WS2812B:WS2812B" V 18125 11125 60  0001 C CNN
@@
 	1    0    0    -1
 $EndComp
-Text GLabel 16950 9175 2    50   Input ~ 0
+Text GLabel 16950 8975 2    50   Input ~ 0
 RGBLED-R
 Wire Wire Line
@@
 Wire Notes Line
 	675  12825 19350 12825
-$Comp
-L Device:R_Small R?
-U 1 1 5EB1E34F
-P 2625 1250
-F 0 "R?" V 2429 1250 50  0000 C CNN
-F 1 "10k" V 2520 1250 50  0000 C CNN
-F 2 "Resistor_SMD:R_0805_2012Metric" H 2625 1250 50  0001 C CNN
-F 3 "~" H 2625 1250 50  0001 C CNN
-	1    2625 1250
-	-1   0    0    1
-$EndComp
-Wire Wire Line
-	2325 1350 2625 1350
-Connection ~ 2625 1350
-Wire Wire Line
-	2625 1350 2900 1350
-$Comp
-L Device:R_Small R?
-U 1 1 5EB22AB3
-P 2625 8825
-F 0 "R?" V 2429 8825 50  0000 C CNN
-F 1 "10k" V 2520 8825 50  0000 C CNN
-F 2 "Resistor_SMD:R_0805_2012Metric" H 2625 8825 50  0001 C CNN
-F 3 "~" H 2625 8825 50  0001 C CNN
-	1    2625 8825
-	-1   0    0    1
-$EndComp
-Connection ~ 2625 8925
-Wire Wire Line
-	2625 8925 2900 8925
 Connection ~ 3400 12225
 Connection ~ 3600 8625
@@
 	1    0    0    -1
 $EndComp
+Wire Wire Line
+	2325 1350 2625 1350
+Wire Wire Line
+	2625 1150 2625 1350
+Connection ~ 2625 1350
+Wire Wire Line
+	2625 1350 2900 1350
+Wire Wire Line
+	2325 8925 2625 8925
+Wire Wire Line
+	2625 8725 2625 8925
+Connection ~ 2625 8925
+Wire Wire Line
+	2625 8925 2900 8925
+$Comp
+L Device:R_Small R91
+U 1 1 5C5D693C
+P 16200 1300
+F 0 "R91" H 16141 1254 50  0000 R CNN
+F 1 "470" H 16141 1345 50  0000 R CNN
+F 2 "Resistor_SMD:R_0805_2012Metric" H 16200 1300 50  0001 C CNN
+F 3 "~" H 16200 1300 50  0001 C CNN
+	1    16200 1300
+	-1   0    0    1
+$EndComp
+$Comp
+L Device:R_Small R92
+U 1 1 5C5DA35E
+P 16950 9075
+F 0 "R92" H 16891 9029 50  0000 R CNN
+F 1 "470" H 16891 9120 50  0000 R CNN
+F 2 "Resistor_SMD:R_0805_2012Metric" H 16950 9075 50  0001 C CNN
+F 3 "~" H 16950 9075 50  0001 C CNN
+	1    16950 9075
+	-1   0    0    1
+$EndComp
 $EndSCHEMATC

Commit message: more traces
Connections:
- net labels added: CAPSLOCK
- wire segments 811 -> 815
Changed lines of the file:
@@
 	-1   0    0    1
 $EndComp
-Wire Wire Line
-	9750 2875 9675 2875
 $Comp
 L MX_Alps_Hybrids:MX-1U MX18
@@
 	9175 2775 9175 3425
 Connection ~ 9175 3425
-Connection ~ 9775 2775
-Connection ~ 9775 3425
-Wire Wire Line
-	9775 3425 9775 2775
 Connection ~ 9775 4075
 Wire Wire Line
@@
 	9525 2725 9825 2725
 Wire Wire Line
-	9475 2775 9775 2775
-Wire Wire Line
-	9375 2875 9675 2875
-Connection ~ 9675 2875
-Wire Wire Line
 	9325 2925 9550 2925
 Connection ~ 9550 2925
@@
 COL8-R
 Wire Wire Line
-	9775 2775 9775 2125
-Connection ~ 9775 2125
-Wire Wire Line
 	9825 2725 9825 2075
 Connection ~ 9825 2075
@@
 	-1   0    0    1
 $EndComp
+Wire Wire Line
+	9375 2875 9675 2875
+Connection ~ 9675 2875
+Wire Wire Line
+	9750 2875 9675 2875
+Wire Wire Line
+	9475 2775 9775 2775
+Text GLabel 9900 2775 2    50   Input ~ 0
+CAPSLOCK
+Wire Wire Line
+	9775 2775 9900 2775
+Connection ~ 9775 2775
+Wire Wire Line
+	9775 2125 9775 2650
+Wire Wire Line
+	9775 2650 9875 2650
+Wire Wire Line
+	9875 2650 9875 2825
+Wire Wire Line
+	9875 2825 9775 2825
+Wire Wire Line
+	9775 2825 9775 3425
+Connection ~ 9775 2125
+Connection ~ 9775 3425
+Text GLabel 4175 1850 2    50   Input ~ 0
+CAPSLOCK
 $EndSCHEMATC

Commit message: added more renders, changed pcb layout
Parts:
- MX31: footprint MX_Alps_Hybrid:MXOnly-1.5U-FLIPPED -> MX_Alps_Hybrid:MXOnly-1U
- MX33, MX35: footprint MX_Alps_Hybrid:MXOnly-1.25U -> MX_Alps_Hybrid:MXOnly-1.25U-FLIPPED
- MX34: footprint MX_Alps_Hybrid:MXOnly-1.5U -> MX_Alps_Hybrid:MXOnly-1.25U
Changed lines of the file:
@@
 F 0 "MX33" H 10936 4267 60  0000 C CNN
 F 1 "MXOnly-1U" H 10936 4193 20  0000 C CNN
-F 2 "MX_Alps_Hybrid:MXOnly-1.25U" H 10825 4025 60  0001 C CNN
+F 2 "MX_Alps_Hybrid:MXOnly-1.25U-FLIPPED" H 10825 4025 60  0001 C CNN
 F 3 "" H 10825 4025 60  0001 C CNN
 	1    10850 4050
@@
 F 0 "MX35" H 11536 4267 60  0000 C CNN
 F 1 "MXOnly-1U" H 11536 4193 20  0000 C CNN
-F 2 "MX_Alps_Hybrid:MXOnly-1.25U" H 11425 4025 60  0001 C CNN
+F 2 "MX_Alps_Hybrid:MXOnly-1.25U-FLIPPED" H 11425 4025 60  0001 C CNN
 F 3 "" H 11425 4025 60  0001 C CNN
 	1    11450 4050
@@
 	13375 3425 13375 4925
 Wire Wire Line
-	9525 4025 9825 4025
-Wire Wire Line
-	9475 4075 9775 4075
-Wire Wire Line
-	9325 4225 9550 4225
-Connection ~ 9550 4225
-Wire Wire Line
 	9775 4075 9775 4925
 Wire Wire Line
-	9375 4175 9675 4175
-Wire Wire Line
 	9750 4175 9675 4175
-Connection ~ 9675 4175
-Connection ~ 9825 4025
 $Comp
 L MX_Alps_Hybrids:MX-1U MX32
@@
 L MX_Alps_Hybrids:MX-1U MX31
 U 1 1 5CCB7222
-P 9350 4050
-F 0 "MX31" H 9436 4267 60  0000 C CNN
-F 1 "MXOnly-1U" H 9436 4193 20  0000 C CNN
-F 2 "MX_Alps_Hybrid:MXOnly-1.5U-FLIPPED" H 9325 4025 60  0001 C CNN
-F 3 "" H 9325 4025 60  0001 C CNN
-	1    9350 4050
+P 10550 4050
+F 0 "MX31" H 10636 4267 60  0000 C CNN
+F 1 "MXOnly-1U" H 10636 4193 20  0000 C CNN
+F 2 "MX_Alps_Hybrid:MXOnly-1U" H 10525 4025 60  0001 C CNN
+F 3 "" H 10525 4025 60  0001 C CNN
+	1    10550 4050
 	1    0    0    -1
 $EndComp
@@
 F 0 "MX34" H 11236 4267 60  0000 C CNN
 F 1 "MXOnly-1U" H 11236 4193 20  0000 C CNN
-F 2 "MX_Alps_Hybrid:MXOnly-1.5U" H 11125 4025 60  0001 C CNN
+F 2 "MX_Alps_Hybrid:MXOnly-1.25U" H 11125 4025 60  0001 C CNN
 F 3 "" H 11125 4025 60  0001 C CNN
 	1    11150 4050
@@
 Text GLabel 4175 1850 2    50   Input ~ 0
 CAPSLOCK
+Wire Wire Line
+	10725 4025 11025 4025
+Connection ~ 11025 4025
+Wire Wire Line
+	10675 4075 10975 4075
+Wire Wire Line
+	10575 4175 10875 4175
+Connection ~ 10875 4175
+Wire Wire Line
+	10525 4225 10750 4225
+Connection ~ 10750 4225
 $EndSCHEMATC

Commit message: removed underglow and backlight, routed left hand
Parts:
- removed C15, C16, C17, C18, C19, C20, C21, C22, C23, C24, C25, C26, C27, C28, C29, C30: 0.1uF, Capacitor_SMD:C_0603_1608Metric, symbol Device:C_Small
- removed LED1, LED10, LED11, LED12, LED13, LED14, LED15, LED16, LED2, LED3, LED4, LED5, LED6, LED7, LED8, LED9: WS2812B, WS2812B:WS2812B, symbol ws2812b:WS2812B
- removed Q1, Q2: 2N7002, Package_TO_SOT_SMD:SOT-23, symbol Transistor_FET:2N7002
- removed R0, R1, R10, R11, R12, R13, R14, R15, R16, R17, R19, R2, R20, R21, R22, R23, R25, R26, R27, R28, R29, R3, R30, R31, R32, R33, R34, R35, R36, R4, R43, R44, R45, R46, R47, R48, R49, R5, R50, R51, R52, R53, R54, R55, R56, R57, R58, R59, R6, R60, R61, R62, R63, R64, R65, R66, R67, R68, R7, R70, R71, R72, R73, R74, R75, R76, R77, R78, R79, R80, R81, R82, R83, R84, R91, R92: 470, Resistor_SMD:R_0805_2012Metric, symbol Device:R_Small
- removed R37, R85: 1k, Resistor_SMD:R_0805_2012Metric, symbol Device:R_Small
- removed SW1, SW2: SW_Push, locallib:SKQGADE010, symbol Switch:SW_Push
- MX0, MX1, MX10, MX11, MX12, MX13, MX14, MX15, MX18, MX19, MX2, MX20, MX21, MX22, MX23, MX25, MX26, MX27, MX28, MX29, MX3, MX30, MX31, MX38, MX39, MX4, MX40, MX41, MX42, MX43, MX44, MX46, MX47, MX48, MX49, MX5, MX50, MX51, MX52, MX53, MX54, MX56, MX57, MX58, MX59, MX6, MX60, MX61, MX62, MX64, MX65, MX66, MX67, MX68, MX69, MX7, MX71, MX72, MX8, MX80, MX81, MX82: value MXOnly-1U -> MXOnly-1U-NoLED; footprint MX_Alps_Hybrid:MXOnly-1U -> MX_Alps_Hybrid:MXOnly-1U-NoLED
- MX16, MX17: value MXOnly-1U -> MXOnly-1U-NoLED
- MX24, MX63, MX74: value MXOnly-1U -> MXOnly-1U-NoLED; footprint MX_Alps_Hybrid:MXOnly-2.25U -> MX_Alps_Hybrid:MXOnly-2.25U-NoLED
- MX32, MX34, MX75, MX77: value MXOnly-1U -> MXOnly-1U-NoLED; footprint MX_Alps_Hybrid:MXOnly-1.25U -> MX_Alps_Hybrid:MXOnly-1.25U-NoLED
- MX33, MX35, MX79: value MXOnly-1U -> MXOnly-1U-NoLED; footprint MX_Alps_Hybrid:MXOnly-1.25U-FLIPPED -> MX_Alps_Hybrid:MXOnly-1.25U-NoLED
- MX36, MX73: value MXOnly-1U -> MXOnly-1U-NoLED; footprint MX_Alps_Hybrid:MXOnly-3U -> MX_Alps_Hybrid:MXOnly-3U-NoLED
- MX37: value MXOnly-1U -> MXOnly-1U-NoLED; footprint MX_Alps_Hybrid:MXOnly-2.75U-FLIPPED -> MX_Alps_Hybrid:MXOnly-2.75U-NoLED
- MX45: value MXOnly-1U -> MXOnly-1U-NoLED; footprint MX_Alps_Hybrid:MXOnly-2U -> MX_Alps_Hybrid:MXOnly-2U-NoLED
- MX55, MX76, MX78, MX9: value MXOnly-1U -> MXOnly-1U-NoLED; footprint MX_Alps_Hybrid:MXOnly-1.5U -> MX_Alps_Hybrid:MXOnly-1.5U-NoLED
- MX70: value MXOnly-1U -> MXOnly-1U-NoLED; footprint MX_Alps_Hybrid:MXOnly-1.75U -> MX_Alps_Hybrid:MXOnly-1.75U-NoLED
Connections:
- net labels removed: LEDGND, LEDGND-R, LEDPWM, LEDPWM-R, RGBLED, RGBLED-R
- wire segments 815 -> 403
- no-connect marks 20 -> 19
Other:
- note removed: "Backlight Control"
