File: pcb/split_65.sch (KiCad schematic (older format))
At the start: 221 parts, among them J1 PJ-3200B-4A, J10 AVR-ISP-6, J11 Breakaway_Tabs, J12 Breakaway_Tabs, J13 Breakaway_Tabs, J14 Breakaway_Tabs, J15 Breakaway_Tabs, J16 Breakaway_Tabs, J2 AVR-ISP-6, J3 Breakaway_Tabs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

Commit message: routed right hand side
Changed lines of the file:
@@
 Wire Wire Line
 	3225 14875 3275 14875
+Text GLabel 4100 9325 2    50   Input ~ 0
+COL0-R
+Text GLabel 4100 9425 2    50   Input ~ 0
+COL1-R
+Text GLabel 4100 9525 2    50   Input ~ 0
+COL2-R
+Text GLabel 4100 9825 2    50   Input ~ 0
+COL3-R
+Text GLabel 4100 9925 2    50   Input ~ 0
+COL4-R
 Text GLabel 4100 10525 2    50   Input ~ 0
-COL0-R
+COL5-R
+Wire Wire Line
+	4500 11025 4100 11025
 Text GLabel 4100 10725 2    50   Input ~ 0
-COL1-R
+COL6-R
+Text GLabel 4100 11125 2    50   Input ~ 0
+ROW0-R
+Text GLabel 4100 11325 2    50   Input ~ 0
+ROW1-R
 Text GLabel 4100 11425 2    50   Input ~ 0
-COL2-R
-Text GLabel 4100 11325 2    50   Input ~ 0
-COL3-R
-Text GLabel 4100 11525 2    50   Input ~ 0
-COL4-R
-Text GLabel 4100 11625 2    50   Input ~ 0
-COL5-R
-Wire Wire Line
-	4500 11025 4100 11025
-Text GLabel 4100 9825 2    50   Input ~ 0
-COL6-R
-Text GLabel 4100 9525 2    50   Input ~ 0
-ROW0-R
-Text GLabel 4100 9425 2    50   Input ~ 0
-ROW1-R
-Text GLabel 4100 9325 2    50   Input ~ 0
 ROW2-R
+Text GLabel 4100 11825 2    50   Input ~ 0
+ROW3-R
 Text GLabel 4100 10825 2    50   Input ~ 0
-ROW3-R
-Text GLabel 4100 11125 2    50   Input ~ 0
 ROW4-R
 Wire Notes Line
@@
 	1    0    0    -1
 $EndComp
-Text GLabel 4175 10425 2    50   Input ~ 0
+Text GLabel 4100 10425 2    50   Input ~ 0
 COL7-R
-Text GLabel 4175 10325 2    50   Input ~ 0
+Text GLabel 4100 10325 2    50   Input ~ 0
 COL8-R
 Wire Wire Line

Commit message: added step files, combined and panelized
Parts:
- removed J15, J16: Breakaway_Tabs, locallib:breakaway-mousebites, symbol Connector_Generic:Conn_01x01
Connections:
- no-connect marks 19 -> 17
Changed lines of the file:
@@
 L Connector_Generic:Conn_01x01 J8
 U 1 1 5BC3C176
-P 6975 7175
-F 0 "J8" H 7054 7217 50  0000 L CNN
-F 1 "Breakaway_Tabs" H 7054 7126 50  0000 L CNN
-F 2 "locallib:breakaway-mousebites" H 6975 7175 50  0001 C CNN
-F 3 "~" H 6975 7175 50  0001 C CNN
-	1    6975 7175
-	1    0    0    -1
-$EndComp
-NoConn ~ 6775 7175
+P 6025 14900
+F 0 "J8" H 6104 14942 50  0000 L CNN
+F 1 "Breakaway_Tabs" H 6104 14851 50  0000 L CNN
+F 2 "locallib:breakaway-mousebites" H 6025 14900 50  0001 C CNN
+F 3 "~" H 6025 14900 50  0001 C CNN
+	1    6025 14900
+	1    0    0    -1
+$EndComp
+NoConn ~ 5825 14900
 NoConn ~ 6775 7000
 Wire Wire Line
@@
 	1    0    0    -1
 $EndComp
-$Comp
-L Connector_Generic:Conn_01x01 J15
-U 1 1 5BCD1D50
-P 6000 14750
-F 0 "J15" H 6079 14792 50  0000 L CNN
-F 1 "Breakaway_Tabs" H 6079 14701 50  0000 L CNN
-F 2 "locallib:breakaway-mousebites" H 6000 14750 50  0001 C CNN
-F 3 "~" H 6000 14750 50  0001 C CNN
-	1    6000 14750
-	1    0    0    -1
-$EndComp
-NoConn ~ 5800 14750
 NoConn ~ 5800 14575
 $Comp
@@
 	1    0    0    -1
 $EndComp
-$Comp
-L Connector_Generic:Conn_01x01 J16
-U 1 1 5BCD1D70
-P 6975 14750
-F 0 "J16" H 7054 14792 50  0000 L CNN
-F 1 "Breakaway_Tabs" H 7054 14701 50  0000 L CNN
-F 2 "locallib:breakaway-mousebites" H 6975 14750 50  0001 C CNN
-F 3 "~" H 6975 14750 50  0001 C CNN
-	1    6975 14750
-	1    0    0    -1
-$EndComp
-NoConn ~ 6775 14750
 NoConn ~ 6775 14575
 Text Notes 13050 7650 0    50   ~ 10
